File: pcb/robohub_prototype_v1/robohub_prototype_v1_uart.kicad_sch (KiCad schematic)
At the start: 13 parts, among them J71 USB_A, U71 MCP2200-I-SO, Y71 Resonator_Small

Commit message: Update paths for footprints top adjacent lib directory at above clone. Finish basic regulator layout/BOM. Link 3d STEPs into model. Rearrangle layout
Parts:
- J71: footprint (none) -> Connector_USB:USB_A_Molex_67643_Horizontal
Changed lines of the file:
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@@
 			)
 		)
-		(property "Footprint" ""
+		(property "Footprint" "Connector_USB:USB_A_Molex_67643_Horizontal"
 			(at 31.75 73.66 0)
 			(effects
