File: pcb/robohub_prototype_v1/robohub_prototype_v1_05212024.kicad_pcb (KiCad board)
At the start: 10 copper layers, 102 parts, among them J21 Barrel_Jack_Switch_Pin3Ring, J51 USB_A, J52 USB_A, J71 USB_A, U1 ATSAMA5D27C, U21 LM3880, U22 TPS564242DRL, U23 TPS564242DRL, U24 TPS564242DRL, U25 TPS564242DRL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

Commit message: Attempts to route ddr
Routing:
- net /DDR2_3/DDR_CS: track 26.4 -> 8.31 mm
- net /DDR2_3/DDR_A10: track 22.4 -> 6.56 mm
- net /DDR2_3/DDR_A0: track 25.1 -> 10.8 mm
- net /DDR2_3/DDR_A4: track 19.7 -> 6.52 mm, vias 2 -> 1
- net /DDR2_3/DDR_A7: track 2.73 -> 14.5 mm
- net /DDR2_3/DDR_A13: track 2.42 -> 13.1 mm
- net /DDR2_3/DDR_D18: track 0.62 -> 9.38 mm
- net /DDR2_3/DDR_A8: track 19.2 -> 12.0 mm
- net /DDR2_3/DDR_BA0: track 3.34 -> 9.44 mm
- net /DDR2_3/DDR_A9: track 2.78 -> 7.69 mm
- net /DDR2_3/DDR_CAS: track 6.50 -> 10.3 mm
- net /DDR2_3/DDR_A12: track 2.08 -> 5.63 mm
- net /DDR2_3/DDR_A5: track 3.28 -> 6.77 mm
- net /DDR2_3/DDR_CLK+: track 4.76 -> 1.53 mm
- net /DDR2_3/DDR_RAS: track 2.25 -> 5.29 mm, vias 2 -> 1
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