File: pcb/robohub_prototype_v1/robohub_prototype_v1_05272024.kicad_pcb (KiCad board)
At the start: 10 copper layers, 102 parts, among them J21 Barrel_Jack_Switch_Pin3Ring, J51 USB_A, J52 USB_A, J71 USB_A, U1 ATSAMA5D27C, U21 LM3880, U22 TPS564242DRL, U23 TPS564242DRL, U24 TPS564242DRL, U25 TPS564242DRL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

Commit message: Attempts to route the ddr2
Parts:
- moved U1 3.34 mm to (121.9, 91.4)
Routing:
- net /DDR2_3/DDR_RAS: track 26.7 -> 0.65 mm, vias 3 -> 1
- net /DDR2_3/DDR_CS: track 26.4 -> 0.94 mm, vias 2 -> 1
- net /DDR2_3/DDR_A7: track 25.5 -> 0.61 mm, vias 2 -> 1
- net /DDR2_3/DDR_A0: track 25.1 -> 0.58 mm, vias 2 -> 1
- net /DDR2_3/DDR_A5: track 23.5 -> 0.70 mm, vias 2 -> 1
- net /DDR2_3/DDR_A13: track 23.3 -> 0.57 mm, vias 2 -> 1
- net /DDR2_3/DDR_A10: track 22.4 -> 0.61 mm, vias 2 -> 1
- net /DDR2_3/DDR_A9: track 21.2 -> 0.59 mm, vias 2 -> 1
- net /DDR2_3/DDR_A8: track 21.0 -> 0.61 mm, vias 2 -> 1
- net /DDR2_3/DDR_A3: track 19.2 -> 2.08 mm, vias 3 -> 0
- net /DDR2_3/DDR_CLK+: track 4.07 -> 19.2 mm
- net /DDR2_3/DDR_A2: track 6.91 -> 21.4 mm, vias 1 -> 0
- net /DDR2_3/DDR_CLK-: track 4.09 -> 18.1 mm
- net /DDR2_3/DDR_CAS: track 11.2 -> 0.60 mm, vias 2 -> 1
- net /DDR2_3/DDR_BA1: track 9.94 -> 0.58 mm, vias 2 -> 1
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