File: pcb/robohub_prototype_v1/robohub_prototype_v1_05282024.kicad_pcb (KiCad board)
At the start: 10 copper layers, 102 parts, among them J21 Barrel_Jack_Switch_Pin3Ring, J51 USB_A, J52 USB_A, J71 USB_A, U1 ATSAMA5D27C, U21 LM3880, U22 TPS564242DRL, U23 TPS564242DRL, U24 TPS564242DRL, U25 TPS564242DRL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

Commit message: Effort at routing ACC
Routing:
- net /DDR2_3/DDR_BA1: track 0.58 -> 29.3 mm, vias 1 -> 2
- net /DDR2_3/DDR_A0: track 0.58 -> 29.0 mm, vias 1 -> 2
- net /DDR2_3/DDR_BA0: track 0.59 -> 29.0 mm, vias 1 -> 3
- net /DDR2_3/DDR_RAS: track 0.65 -> 28.9 mm, vias 1 -> 2
- net /DDR2_3/DDR_A5: track 0.70 -> 28.9 mm, vias 1 -> 2
- net /DDR2_3/DDR_A9: track 0.59 -> 28.7 mm, vias 1 -> 2
- net /DDR2_3/DDR_A6: track 0.60 -> 28.5 mm, vias 1 -> 2
- net /DDR2_3/DDR_A8: track 0.61 -> 28.5 mm, vias 1 -> 2
- net /DDR2_3/DDR_A10: track 0.61 -> 28.4 mm, vias 1 -> 2
- net /DDR2_3/DDR_CAS: track 0.60 -> 28.2 mm, vias 1 -> 2
- net /DDR2_3/DDR_CS: track 0.94 -> 28.4 mm, vias 1 -> 2
- net /DDR2_3/DDR_A7: track 0.61 -> 28.0 mm, vias 1 -> 2
- net /DDR2_3/DDR_WE: track 0.66 -> 27.9 mm, vias 1 -> 2
- net /DDR2_3/DDR_A13: track 0.57 -> 27.8 mm, vias 1 -> 2
- net /DDR2_3/DDR_A3: track 2.08 -> 28.5 mm, vias 0 -> 2
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