File: pcb/robohub_prototype_v1/robohub_prototype_v1_sdcard.kicad_sch (KiCad schematic)
At the start: 9 parts, among them U61 molex_5025700893

Commit message: Update paths to footprint libraries. Begin adding footprints for PDN resistors. Create master BOM
Parts:
- U61: footprint custom_footprint:molex_5025700893 -> fryelabs:molex_5025700893
Changed lines of the file:
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@@
 			)
 		)
-		(property "Footprint" "custom_footprint:molex_5025700893"
+		(property "Footprint" "fryelabs:molex_5025700893"
 			(at 163.83 78.74 0)
 			(effects

Commit message: Begin PDN circuit design/BOM/layout
Parts:
- U61: footprint fryelabs:molex_5025700893 -> fryelabs_kicad_footprint_lib:molex_5025700893
Changed lines of the file:
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@@
 			)
 		)
-		(property "Footprint" "fryelabs:molex_5025700893"
+		(property "Footprint" "fryelabs_kicad_footprint_lib:molex_5025700893"
 			(at 163.83 78.74 0)
 			(effects

Commit message: Update footprint assignment. begin laying out ethernet
Parts:
- C61: footprint (none) -> Capacitor_SMD:C_0402_1005Metric
Changed lines of the file:
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@@
 			)
 		)
-		(property "Footprint" ""
+		(property "Footprint" "Capacitor_SMD:C_0402_1005Metric"
 			(at 28.9052 149.86 0)
 			(effects
