File: pcb/robohub_prototype_v1/robohub_prototype_v1_usb.kicad_sch (KiCad schematic)
At the start: 6 parts, among them J51 USB_A, J52 USB_A

Commit message: Update footprint assignment. begin laying out ethernet
Parts:
- FB51: footprint (none) -> Resistor_SMD:R_0402_1005Metric
Changed lines of the file:
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@@
 			)
 		)
-		(property "Footprint" ""
+		(property "Footprint" "Resistor_SMD:R_0402_1005Metric"
 			(at 228.6 36.068 90)
 			(effects
